File: hardware/motherboard_rev1.sch (EAGLE design)
At the start: 81 parts, among them CN1 UG-2828GDEDF11-1.5OLED, CN2 1X05, CN3 1X06, CN4 FEMALE, CN6 CON-MOLEX-2MMFEMALE, CN7 CON-MOLEX-2MMFEMALE_RA, CN8 CON-MOLEX-2MMFEMALE_RA, CN9 CON-MOLEX-2MMFEMALE_RA, U1 MCP73831, X1 CRYSTAL-ABM7-8.000MHZ-D-2-Y-T

Commit message: Added revision 1 to motherboard, as well as CHANGELOG file
Parts:
- removed TP1, TP2: TEST-POINT2, SparkFun-Passives:TEST-POINT2
- added R16, R17: 4.7k, notes_mark5a:RESISTOR0603
- CN3: value 1X06 -> PHF-106-01-L-S
Connections:
- net 3.3V: now also C1.1, C12.2, C8.2, L1.2, R16.2, R17.2, U$24.VIN, U$3.VDD2, U$3.VDD5; no longer C12.1, C8.1, TP1.1, TP2.1, U$3.VSS1, U$3.VSS4
- net GND: now also C12.1, C8.1, U$3.VSS1, U$3.VSS4; no longer C12.2, C8.2, U$3.VDD2, U$3.VDD5
- net SCL1: now also R17.1
- net SDA1: now also R16.1
- net VIN: no longer C1.1, L1.2, U$24.VIN
Other:
- note added: "I2C PULL-UP"
- note added: "Revision 1 (Oct 2014)"
- note removed: "Revision 0 (July 2014)"
