File: hardware/touch_rev2.brd (EAGLE design)
At the start: 39.5 x 54 mm, 17 parts, among them SW1 SWITCH, SW2 SWITCH, U1 MPR121-TOUCH-CONTROLLER, U2 M41T82ZM6F, U3 CAPACITIVE-WHEEL-8, X1 32.768kHz

Commit message: Added motherboard rev1 and capacitive touch board rev2
Routing:
- net GND: track 0.00 -> 1.16 mm
Other:
- outline, holes or cut-outs redrawn
- board text removed: "Arducorder"
- board text removed: "Mini"
- board text removed: "OSH"
- board text removed: "rev1"
Changed lines of the file:
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@@
 <setting verticaltext="up"/>
 </settings>
-<grid distance="0.25" unitdist="mm" unit="mm" style="lines" multiple="1" display="yes" altdistance="0.025" altunitdist="inch" altunit="inch"/>
+<grid distance="1" unitdist="mil" unit="mil" style="lines" multiple="1" display="yes" altdistance="0.025" altunitdist="inch" altunit="inch"/>
 <layers>
 <layer number="1" name="Top" color="4" fill="1" visible="yes" active="yes"/>
@@
 <board>
 <plain>
-<wire x1="50.25" y1="5.75" x2="89.75" y2="5.75" width="0" layer="20"/>
+<wire x1="50.25" y1="5.75" x2="56.75" y2="5.75" width="0" layer="20"/>
+<wire x1="56.75" y1="5.75" x2="62" y2="11" width="0" layer="20"/>
+<wire x1="62" y1="11" x2="78" y2="11" width="0" layer="20"/>
+<wire x1="78" y1="11" x2="83.25" y2="5.75" width="0" layer="20"/>
+<wire x1="83.25" y1="5.75" x2="89.75" y2="5.75" width="0" layer="20"/>
 <wire x1="89.75" y1="5.75" x2="89.75" y2="58.75" width="0" layer="20"/>
 <wire x1="89.75" y1="58.75" x2="88.75" y2="59.75" width="0" layer="20"/>
@@
 <rectangle x1="53" y1="22" x2="61" y2="28" layer="40"/>
 <rectangle x1="55" y1="28.5" x2="70.5" y2="41.5" layer="40"/>
-<text x="60.5" y="94.25" size="1.016" layer="22" rot="MR0">Arducorder</text>
-<text x="60.5" y="92.75" size="1.016" layer="22" rot="MR0">Mini</text>
-<text x="60.5" y="91.25" size="1.016" layer="22" rot="MR0">rev1</text>
 <text x="52.75" y="13.5" size="1.778" layer="21" rot="R90">make | share | dream | give</text>
-<wire x1="68.625" y1="79.875" x2="71.375" y2="79.875" width="0.2032" layer="22" curve="-247.380135"/>
-<wire x1="71.375" y1="79.875" x2="71.875" y2="78.625" width="0.2032" layer="22"/>
-<wire x1="68.625" y1="79.875" x2="68.125" y2="78.625" width="0.2032" layer="22"/>
-<wire x1="68.125" y1="78.625" x2="67.75" y2="79" width="0.2032" layer="22"/>
-<wire x1="67.75" y1="79" x2="67" y2="78.5" width="0.2032" layer="22"/>
-<wire x1="67" y1="78.5" x2="66.5" y2="79" width="0.2032" layer="22"/>
-<wire x1="66.5" y1="79" x2="67" y2="79.75" width="0.2032" layer="22"/>
-<wire x1="71.875" y1="78.625" x2="72.25" y2="79" width="0.2032" layer="22"/>
-<wire x1="72.25" y1="79" x2="73" y2="78.5" width="0.2032" layer="22"/>
-<wire x1="73" y1="78.5" x2="73.5" y2="79" width="0.2032" layer="22"/>
-<wire x1="73.5" y1="79" x2="73" y2="79.75" width="0.2032" layer="22"/>
-<wire x1="66.75" y1="80.75" x2="66" y2="81" width="0.2032" layer="22"/>
-<wire x1="66" y1="81" x2="66" y2="81.625" width="0.2032" layer="22"/>
-<wire x1="66" y1="81.625" x2="66.75" y2="81.875" width="0.2032" layer="22"/>
-<wire x1="73.25" y1="80.75" x2="74" y2="81" width="0.2032" layer="22"/>
-<wire x1="74" y1="81" x2="74" y2="81.625" width="0.2032" layer="22"/>
-<wire x1="74" y1="81.625" x2="73.25" y2="81.875" width="0.2032" layer="22"/>
-<wire x1="69.375" y1="84.25" x2="69.625" y2="85" width="0.2032" layer="22"/>
-<wire x1="69.625" y1="85" x2="70.375" y2="85" width="0.2032" layer="22"/>
-<wire x1="70.375" y1="85" x2="70.625" y2="84.25" width="0.2032" layer="22"/>
-<wire x1="67.25" y1="83" x2="67" y2="83.75" width="0.2032" layer="22"/>
-<wire x1="67" y1="83.75" x2="67.5" y2="84.25" width="0.2032" layer="22"/>
-<wire x1="67.5" y1="84.25" x2="68.25" y2="83.75" width="0.2032" layer="22"/>
-<wire x1="72.75" y1="83" x2="73" y2="83.75" width="0.2032" layer="22"/>
-<wire x1="73" y1="83.75" x2="72.5" y2="84.25" width="0.2032" layer="22"/>
-<wire x1="72.5" y1="84.25" x2="71.75" y2="83.75" width="0.2032" layer="22"/>
-<wire x1="73.25" y1="80.75" x2="73" y2="79.75" width="0.2032" layer="22" curve="-17.818889"/>
-<wire x1="72.75" y1="83" x2="73.25" y2="81.875" width="0.2032" layer="22" curve="-24.227745"/>
-<wire x1="70.625" y1="84.25" x2="71.75" y2="83.75" width="0.2032" layer="22" curve="-24.227745"/>
-<wire x1="68.25" y1="83.75" x2="69.375" y2="84.25" width="0.2032" layer="22" curve="-24.599791"/>
-<wire x1="66.75" y1="81.875" x2="67.25" y2="83" width="0.2032" layer="22" curve="-24.599791"/>
-<wire x1="67" y1="79.75" x2="66.75" y2="80.75" width="0.2032" layer="22" curve="-18.717192"/>
-<text x="71.625" y="78" size="1.016" layer="22" rot="MR0">OSH</text>
 <circle x="53.25" y="56" radius="2" width="0.1778" layer="21"/>
 <circle x="53.25" y="56" radius="2.06155" width="0.1778" layer="22"/>
@@
 <circle x="87.5" y="8.5" radius="2.06155" width="0.1778" layer="22"/>
 <circle x="52.5" y="8.5" radius="2.06155" width="0.1778" layer="22"/>
-<wire x1="48" y1="11" x2="62" y2="11" width="0.2032" layer="21"/>
-<wire x1="62" y1="11" x2="78" y2="11" width="0.2032" layer="21"/>
-<wire x1="78" y1="11" x2="92" y2="11" width="0.2032" layer="21"/>
-<wire x1="83" y1="6" x2="78" y2="11" width="0.2032" layer="21"/>
-<wire x1="57" y1="6" x2="62" y2="11" width="0.2032" layer="21"/>
 <wire x1="74.5" y1="23.25" x2="75" y2="23.25" width="0.1778" layer="21"/>
 <wire x1="74.75" y1="23.5" x2="74.75" y2="23" width="0.1778" layer="21"/>
@@
 <param name="mdWirePad" value="7mil"/>
 <param name="mdWireVia" value="7mil"/>
-<param name="mdPadPad" value="7mil"/>
+<param name="mdPadPad" value="6mil"/>
 <param name="mdPadVia" value="7mil"/>
 <param name="mdViaVia" value="7mil"/>
@@
 <via x="78.5" y="25.5" extent="1-16" drill="0.3302"/>
 <via x="78.5" y="21" extent="1-16" drill="0.3302"/>
+<wire x1="63.1444" y1="21.8186" x2="63.8048" y2="21.8186" width="0.1778" layer="16"/>
+<wire x1="63.8048" y1="21.8186" x2="64.1604" y2="22.1742" width="0.1778" layer="16"/>
+<wire x1="63.1444" y1="21.8186" x2="63.15" y2="21.825" width="0" layer="19" extent="16-16"/>
 </signal>
 <signal name="3.3V">
@@
 <contactref element="U1" pad="9"/>
 <contactref element="U3" pad="7"/>
-<wire x1="63.15" y1="23.025" x2="63.125" y2="23" width="0.2032" layer="16"/>
-<wire x1="63.125" y1="23" x2="61.75" y2="23" width="0.2032" layer="16"/>
-<wire x1="61.75" y1="23" x2="60.5" y2="24.25" width="0.2032" layer="16"/>
+<wire x1="63.15" y1="23.025" x2="63.125" y2="23.0254" width="0.2032" layer="16"/>
+<wire x1="63.125" y1="23.0254" x2="61.7246" y2="23.0254" width="0.2032" layer="16"/>
+<wire x1="61.7246" y1="23.0254" x2="60.5" y2="24.25" width="0.2032" layer="16"/>
 <wire x1="60.5" y1="24.25" x2="60.5" y2="32.25" width="0.2032" layer="16"/>
 <wire x1="60.5" y1="32.25" x2="54.875" y2="37.875" width="0.2032" layer="16"/>
